File: MP1584_TRYOUT.sch (KiCad schematic (older format))
At the start: 15 parts

Commit message: update,
Parts:
- removed D?: SD_1N5822_SS34, w_smd_diode:do214aa, symbol taobao-sd:SD_1N5822_SS34
- removed J?: Conn_01x03_Female, Connector_PinHeader_1.27mm:PinHeader_1x03_P1.27mm_Vertical, symbol Connector:Conn_01x03_Female
- added D5: D_1N4148_T4, Diode_SMD:D_SOD-123, symbol taobao-d:D_1N4148_T4
- added J6, J7: Conn_01x03_Female, Connector_PinHeader_2.54mm:PinHeader_1x02_P2.54mm_Vertical, symbol Connector:Conn_01x02_Female
- gave numbers to parts that had none: 13
Connections:
- net +5V: now also J7.1 (Pin_1)
- net GND: now also D5.2 (A), J6.2 (Pin_2), J7.2 (Pin_2)
- net at C1.1, L1.1, U5.1 (SW): now also D5.1 (K)
- net PWR: now reaches C2.1, R9.1, U5.7 (VIN)
- net PWR: now also J6.1 (Pin_1)

Commit message: DRC ok,
Parts:
- J6: value Conn_01x03_Female -> POWER_IN
- J7: value Conn_01x03_Female -> POWER_OUT
Changed lines of the file:
@@
 AR Path="/5CE35579/5CDF3426" Ref="R13"  Part="1"
 AR Path="/5CE8687D/5CDF3426" Ref="R?"  Part="1"
-F 0 "R13" H 7500 3900 50  0000 L CNN
-F 1 "R433,0603" H 7500 3850 50  0000 L CNN
+F 0 "R13" H 7300 3900 50  0000 R CNN
+F 1 "R433,0603" H 7300 3850 50  0000 R CNN
 F 2 "Resistor_SMD:R_0603_1608Metric_Pad1.05x0.95mm_HandSolder" H 7400 3850 50  0001 C CNN
 F 3 "~" H 7400 3850 50  0001 C CNN
@@
 AR Path="/5CE35579/5CEA5AA1" Ref="J7"  Part="1"
 AR Path="/5CE8687D/5CEA5AA1" Ref="J?"  Part="1"
-F 0 "J7" H 9250 3100 50  0000 C CNN
-F 1 "Conn_01x03_Female" H 9250 3200 50  0000 C CNN
+F 0 "J7" H 9450 3450 50  0000 L CNN
+F 1 "POWER_OUT" H 9450 3350 50  0000 L CNN
 F 2 "Connector_PinHeader_2.54mm:PinHeader_1x02_P2.54mm_Vertical" H 9400 3450 50  0001 C CNN
 F 3 "~" H 9400 3450 50  0001 C CNN
@@
 AR Path="/5CE8687D/5CEA78ED" Ref="#PWR?"  Part="1"
 F 0 "#PWR0101" H 9100 3400 50  0001 C CNN
-F 1 "GND" H 9150 3450 50  0000 C CNN
+F 1 "GND" H 9000 3650 50  0000 R CNN
 F 2 "" H 9100 3650 50  0001 C CNN
 F 3 "" H 9100 3650 50  0001 C CNN
@@
 AR Path="/5CE8687D/5CEABA63" Ref="J?"  Part="1"
 F 0 "J6" H 2350 2850 50  0000 C CNN
-F 1 "Conn_01x03_Female" H 2350 2950 50  0000 C CNN
+F 1 "POWER_IN" H 2350 2950 50  0000 C CNN
 F 2 "Connector_PinHeader_2.54mm:PinHeader_1x02_P2.54mm_Vertical" H 2500 3200 50  0001 C CNN
 F 3 "~" H 2500 3200 50  0001 C CNN

Commit message: update led on MP1584 and DRC ok,
Parts:
- added D6: LED_GREEN,0805, footprint-lib:LED_0805_2012Metric, symbol taobao-led:LED_GREEN,0805
- added R15: R103,0805, Resistor_SMD:R_0805_2012Metric_Pad1.15x1.40mm_HandSolder, symbol taobao-r:R103,0805
Connections:
- net GND: now also R15.2
- net +5V: no longer names the net of C4.1, C5.1, J7.1 (Pin_1), L1.2, R10.1
- net +5V: now also D6.2 (A)
- new net: D6.1 (K), R15.1
Other:
- moved on the sheet: J7
Changed lines of the file:
@@
 Connection ~ 8550 4100
-$Comp
-L power:+5V #PWR04
-U 1 1 5CE1355F
-P 8750 3150
-AR Path="/5CE35579/5CE1355F" Ref="#PWR04"  Part="1"
-AR Path="/5CE8687D/5CE1355F" Ref="#PWR?"  Part="1"
-F 0 "#PWR04" H 8750 3000 50  0001 C CNN
-F 1 "+5V" H 8800 3350 50  0000 C CNN
-F 2 "" H 8750 3150 50  0001 C CNN
-F 3 "" H 8750 3150 50  0001 C CNN
-	1    8750 3150
-	1    0    0    -1
-$EndComp
-Wire Wire Line
-	8750 3150 8750 3350
-Connection ~ 8750 3350
 $Comp
 L power:GND #PWR02
@@
 L Connector:Conn_01x02_Female J7
 U 1 1 5CEA5AA1
-P 9400 3450
+P 10300 3350
 AR Path="/5CE35579/5CEA5AA1" Ref="J7"  Part="1"
 AR Path="/5CE8687D/5CEA5AA1" Ref="J?"  Part="1"
-F 0 "J7" H 9450 3450 50  0000 L CNN
-F 1 "POWER_OUT" H 9450 3350 50  0000 L CNN
-F 2 "Connector_PinHeader_2.54mm:PinHeader_1x02_P2.54mm_Vertical" H 9400 3450 50  0001 C CNN
-F 3 "~" H 9400 3450 50  0001 C CNN
-	1    9400 3450
+F 0 "J7" H 10350 3350 50  0000 L CNN
+F 1 "POWER_OUT" H 10350 3250 50  0000 L CNN
+F 2 "Connector_PinHeader_2.54mm:PinHeader_1x02_P2.54mm_Vertical" H 10300 3350 50  0001 C CNN
+F 3 "~" H 10300 3350 50  0001 C CNN
+	1    10300 3350
 	1    0    0    -1
 $EndComp
@@
 L power:GND #PWR0101
 U 1 1 5CEA78ED
-P 9100 3650
+P 10000 3550
 AR Path="/5CE35579/5CEA78ED" Ref="#PWR0101"  Part="1"
 AR Path="/5CE8687D/5CEA78ED" Ref="#PWR?"  Part="1"
-F 0 "#PWR0101" H 9100 3400 50  0001 C CNN
-F 1 "GND" H 9000 3650 50  0000 R CNN
-F 2 "" H 9100 3650 50  0001 C CNN
-F 3 "" H 9100 3650 50  0001 C CNN
-	1    9100 3650
+F 0 "#PWR0101" H 10000 3300 50  0001 C CNN
+F 1 "GND" H 9900 3550 50  0000 R CNN
+F 2 "" H 10000 3550 50  0001 C CNN
+F 3 "" H 10000 3550 50  0001 C CNN
+	1    10000 3550
 	1    0    0    -1
 $EndComp
 Wire Wire Line
-	9200 3550 9100 3550
+	10100 3450 10000 3450
 Wire Wire Line
-	9100 3550 9100 3650
-$Comp
-L power:+5V #PWR0102
-U 1 1 5CEA8A1D
-P 9100 3350
-AR Path="/5CE35579/5CEA8A1D" Ref="#PWR0102"  Part="1"
-AR Path="/5CE8687D/5CEA8A1D" Ref="#PWR?"  Part="1"
-F 0 "#PWR0102" H 9100 3200 50  0001 C CNN
-F 1 "+5V" H 9150 3550 50  0000 C CNN
-F 2 "" H 9100 3350 50  0001 C CNN
-F 3 "" H 9100 3350 50  0001 C CNN
-	1    9100 3350
-	1    0    0    -1
-$EndComp
-Wire Wire Line
-	9100 3350 9100 3450
-Wire Wire Line
-	9100 3450 9200 3450
+	10000 3450 10000 3550
 $Comp
 L Connector:Conn_01x02_Female J6
@@
 AR Path="/5CE35579/5CEABA63" Ref="J6"  Part="1"
 AR Path="/5CE8687D/5CEABA63" Ref="J?"  Part="1"
-F 0 "J6" H 2350 2850 50  0000 C CNN
-F 1 "POWER_IN" H 2350 2950 50  0000 C CNN
+F 0 "J6" H 2350 3400 50  0000 C CNN
+F 1 "POWER_IN" H 2350 3300 50  0000 C CNN
 F 2 "Connector_PinHeader_2.54mm:PinHeader_1x02_P2.54mm_Vertical" H 2500 3200 50  0001 C CNN
 F 3 "~" H 2500 3200 50  0001 C CNN
@@
 	-1   0    0    -1
 $EndComp
+$Comp
+L taobao-led:LED_GREEN,0805 D?
+U 1 1 5CF154E2
+P 9350 3550
+AR Path="/5CF154E2" Ref="D?"  Part="1"
+AR Path="/5CE35579/5CF154E2" Ref="D6"  Part="1"
+F 0 "D6" V 9400 3450 50  0000 R CNN
+F 1 "LED_GREEN,0805" V 9350 3450 50  0000 R CNN
+F 2 "footprint-lib:LED_0805_2012Metric" V 9350 3550 50  0001 C CNN
+F 3 "" V 9350 3550 50  0001 C CNN
+	1    9350 3550
+	0    -1   -1   0
+$EndComp
+$Comp
+L taobao-r:R103,0805 R?
+U 1 1 5CF154E8
+P 9350 3800
+AR Path="/5CF154E8" Ref="R?"  Part="1"
+AR Path="/5CE35579/5CF154E8" Ref="R15"  Part="1"
+F 0 "R15" H 9450 3850 50  0000 L CNN
+F 1 "R103,0805" H 9450 3800 50  0000 L CNN
+F 2 "Resistor_SMD:R_0805_2012Metric_Pad1.15x1.40mm_HandSolder" H 9350 3800 50  0001 C CNN
+F 3 "~" H 9350 3800 50  0001 C CNN
+	1    9350 3800
+	1    0    0    -1
+$EndComp
+Wire Wire Line
+	9350 3950 9350 3900
+Wire Wire Line
+	9350 3650 9350 3700
+$Comp
+L power:GND #PWR0102
+U 1 1 5CF183D6
+P 9350 3950
+AR Path="/5CE35579/5CF183D6" Ref="#PWR0102"  Part="1"
+AR Path="/5CE8687D/5CF183D6" Ref="#PWR?"  Part="1"
+F 0 "#PWR0102" H 9350 3700 50  0001 C CNN
+F 1 "GND" H 9250 3950 50  0000 R CNN
+F 2 "" H 9350 3950 50  0001 C CNN
+F 3 "" H 9350 3950 50  0001 C CNN
+	1    9350 3950
+	1    0    0    -1
+$EndComp
+Wire Wire Line
+	9350 3450 9350 3350
+Connection ~ 9350 3350
+Wire Wire Line
+	9350 3350 10100 3350
+Connection ~ 8750 3350
+Wire Wire Line
+	8750 3350 9350 3350
 $EndSCHEMATC
