File: power-board-tryout.sch (KiCad schematic (older format))
At the start: 39 parts, among them J1 3V3_OUT, J2 Screw_Terminal_01x04, J3 5V_OUT, J4 AUX1_OUT, J5 AUX2_OUT, J6 AUX3_OUT, U1 MP1584-BREAKOUT-BOARD, U2 MP1584-BREAKOUT-BOARD, U3 MP1584-BREAKOUT-BOARD, U4 MP1584-BREAKOUT-BOARD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

Commit message: update,
Parts:
- removed D5: LED_GREEN,0805, LED_SMD:LED_0805_2012Metric_Pad1.15x1.40mm_HandSolder, symbol taobao-led:LED_GREEN,0805
- removed J6: AUX3_OUT, footprint-lib:PinHeader_1x02_P2.54mm_power_output_terminal, symbol Connector:Conn_01x02_Male
- removed JP8: Jumper_NO_Small, Jumper:SolderJumper-2_P1.3mm_Open_TrianglePad1.0x1.5mm, symbol Device:Jumper_NO_Small
- removed JP9: Jumper_2_Open, Jumper:SolderJumper-2_P1.3mm_Open_TrianglePad1.0x1.5mm, symbol Jumper:Jumper_2_Open
- removed R10: R103,0805, Resistor_SMD:R_0805_2012Metric_Pad1.15x1.40mm_HandSolder, symbol taobao-r:R103,0805
- removed R9: VAR_5V6,0805, footprint-lib:VAR_0805, symbol taobao-varistor:VAR_5V6,0805
- removed U5: MP1584-BREAKOUT-BOARD, footprint-lib:MP1584_buck_module, symbol taobao-board:MP1584-BREAKOUT-BOARD
Changed lines of the file:
@@
 EESchema Schematic File Version 4
 LIBS:power-board-tryout-cache
-LIBS:MP1584-tryout-cache
 EELAYER 29 0
 EELAYER END
@@
 $EndComp
 $Comp
-L taobao-board:MP1584-BREAKOUT-BOARD U5
-U 1 1 5CE2B54C
-P 3500 5300
-F 0 "U5" H 3500 5800 50  0000 C CNN
-F 1 "MP1584-BREAKOUT-BOARD" H 3500 5700 50  0000 C CNN
-F 2 "footprint-lib:MP1584_buck_module" H 3500 5300 50  0001 C CNN
-F 3 "" H 3500 5300 50  0001 C CNN
-	1    3500 5300
-	1    0    0    -1
-$EndComp
-$Comp
 L Jumper:Jumper_2_Open JP1
 U 1 1 5CE2BEEF
@@
 	1    0    0    -1
 $EndComp
-$Comp
-L Jumper:Jumper_2_Open JP9
-U 1 1 5CE2D6EF
-P 4700 5150
-F 0 "JP9" H 4700 5400 50  0000 C CNN
-F 1 "Jumper_2_Open" H 4700 5300 50  0000 C CNN
-F 2 "Jumper:SolderJumper-2_P1.3mm_Open_TrianglePad1.0x1.5mm" H 4700 5150 50  0001 C CNN
-F 3 "~" H 4700 5150 50  0001 C CNN
-	1    4700 5150
-	1    0    0    -1
-$EndComp
 Wire Wire Line
 	4100 1450 4500 1450
@@
 Wire Wire Line
 	4100 4200 4500 4200
-Wire Wire Line
-	4100 5150 4500 5150
 $Comp
 L Connector:Conn_01x02_Male J1
@@
 	4200 4500 4100 4500
 Wire Wire Line
-	4200 5450 4100 5450
-Wire Wire Line
 	2900 1450 2600 1450
 Wire Wire Line
@@
 Connection ~ 2600 3300
 Wire Wire Line
-	2600 4200 2600 5150
-Wire Wire Line
-	2600 5150 2900 5150
-Connection ~ 2600 4200
-Wire Wire Line
-	2900 5450 2800 5450
-Wire Wire Line
-	2800 5450 2800 4500
-Wire Wire Line
 	2800 4500 2900 4500
 Wire Wire Line
@@
 Wire Wire Line
 	2800 3600 2900 3600
-Connection ~ 2800 4500
 Wire Wire Line
 	2800 3600 2800 2700
@@
 PWR
 $Comp
-L power:GND #PWR0101
+L power:GND #PWR01
 U 1 1 5CE3A947
 P 2050 1950
-F 0 "#PWR0101" H 2050 1700 50  0001 C CNN
+F 0 "#PWR01" H 2050 1700 50  0001 C CNN
 F 1 "GND" H 2100 1750 50  0000 C CNN
 F 2 "" H 2050 1950 50  0001 C CNN
@@
 	4200 4500 4200 4450
 $Comp
-L Device:Jumper_NO_Small JP8
-U 1 1 5CE42DAC
-P 4200 4850
-F 0 "JP8" V 4150 4900 50  0000 L CNN
-F 1 "Jumper_NO_Small" V 4200 4900 50  0000 L CNN
-F 2 "Jumper:SolderJumper-2_P1.3mm_Open_TrianglePad1.0x1.5mm" H 4200 4850 50  0001 C CNN
-F 3 "~" H 4200 4850 50  0001 C CNN
-	1    4200 4850
-	0    1    1    0
-$EndComp
-Wire Wire Line
-	4200 4500 4200 4750
-Connection ~ 4200 4500
-Wire Wire Line
-	4200 4950 4200 5400
-$Comp
 L Connector:Conn_01x02_Male J3
 U 1 1 5CE466E7
@@
 $EndComp
 $Comp
-L Connector:Conn_01x02_Male J6
-U 1 1 5CE499FD
-P 6500 5150
-F 0 "J6" H 6450 5150 50  0000 R CNN
-F 1 "AUX3_OUT" H 6450 5050 50  0000 R CNN
-F 2 "footprint-lib:PinHeader_1x02_P2.54mm_power_output_terminal" H 6500 5150 50  0001 C CNN
-F 3 "~" H 6500 5150 50  0001 C CNN
-	1    6500 5150
-	-1   0    0    -1
-$EndComp
-$Comp
 L taobao-led:LED_GREEN,0805 D1
 U 1 1 5CE4AC96
@@
 Wire Wire Line
 	5900 4550 5900 4600
-$Comp
-L taobao-led:LED_GREEN,0805 D5
-U 1 1 5CE6F135
-P 5900 5400
-F 0 "D5" V 5950 5300 50  0000 R CNN
-F 1 "LED_GREEN,0805" V 5900 5300 50  0000 R CNN
-F 2 "LED_SMD:LED_0805_2012Metric_Pad1.15x1.40mm_HandSolder" V 5900 5400 50  0001 C CNN
-F 3 "" V 5900 5400 50  0001 C CNN
-	1    5900 5400
-	0    -1   -1   0
-$EndComp
-$Comp
-L taobao-r:R103,0805 R10
-U 1 1 5CE6F13F
-P 5900 5650
-F 0 "R10" H 6000 5700 50  0000 L CNN
-F 1 "R103,0805" H 6000 5650 50  0000 L CNN
-F 2 "Resistor_SMD:R_0805_2012Metric_Pad1.15x1.40mm_HandSolder" H 5900 5650 50  0001 C CNN
-F 3 "~" H 5900 5650 50  0001 C CNN
-	1    5900 5650
-	1    0    0    -1
-$EndComp
-Wire Wire Line
-	5900 5150 5900 5300
-Wire Wire Line
-	5900 5800 5900 5750
-Wire Wire Line
-	5900 5500 5900 5550
-Wire Wire Line
-	4900 5150 5550 5150
-Connection ~ 5900 5150
-Wire Wire Line
-	5900 5150 6300 5150
 Wire Wire Line
 	4900 4200 5550 4200
@@
 Wire Wire Line
 	4200 4450 4200 4100
-Wire Wire Line
-	4200 5400 5300 5400
-Wire Wire Line
-	5300 5400 5300 5250
-Wire Wire Line
-	5300 5250 6300 5250
-Connection ~ 4200 5400
-Wire Wire Line
-	4200 5400 4200 5450
 $Comp
 L taobao-varistor:VAR_5V6,0805 R1
@@
 Wire Wire Line
 	5550 4200 5900 4200
-$Comp
-L taobao-varistor:VAR_5V6,0805 R9
-U 1 1 5CE45FA9
-P 5550 5500
-F 0 "R9" H 5700 5550 50  0000 L CNN
-F 1 "VAR_5V6,0805" H 5700 5500 50  0000 L CNN
-F 2 "footprint-lib:VAR_0805" H 5550 5500 50  0001 C CNN
-F 3 "~" H 5550 5500 50  0001 C CNN
-	1    5550 5500
-	1    0    0    -1
-$EndComp
-Wire Wire Line
-	5550 5650 5550 5800
-Wire Wire Line
-	5550 5150 5550 5350
-Connection ~ 5550 5150
-Wire Wire Line
-	5550 5150 5900 5150
-Wire Wire Line
-	5900 5800 5550 5800
-Wire Wire Line
-	5550 5800 5300 5800
-Wire Wire Line
-	5300 5800 5300 5400
-Connection ~ 5550 5800
-Connection ~ 5300 5400
 Wire Wire Line
 	5300 4850 5300 4450
@@
 F0 "MP1584_TRYOUT" 50
 F1 "MP1584_TRYOUT.sch" 50
+F2 "PWR" I L 8500 1550 50
 $EndSheet
+Text Label 8000 1550 0    50   ~ 0
+PWR
+Wire Wire Line
+	8500 1550 8000 1550
 $EndSCHEMATC

Commit message: DRC ok,
Changed lines of the file:
@@
 F 0 "J2" H 1250 1950 50  0000 C CNN
 F 1 "Screw_Terminal_01x04" H 1250 1850 50  0000 C CNN
-F 2 "Connector_PinHeader_2.54mm:PinHeader_1x04_P2.54mm_Vertical" H 1350 1600 50  0000 C CNN
+F 2 "Connector_PinHeader_2.54mm:PinHeader_1x04_P2.54mm_Vertical" H 1350 1600 50  0001 C CNN
 F 3 "~" H 1350 1600 50  0001 C CNN
 	1    1350 1600

Commit message: update led on MP1584 and DRC ok,
Parts:
- D1, D2, D3, D4: footprint LED_SMD:LED_0805_2012Metric_Pad1.15x1.40mm_HandSolder -> footprint-lib:LED_0805_2012Metric
Changed lines of the file:
@@
 F 0 "D1" V 5950 1600 50  0000 R CNN
 F 1 "LED_GREEN,0805" V 5900 1600 50  0000 R CNN
-F 2 "LED_SMD:LED_0805_2012Metric_Pad1.15x1.40mm_HandSolder" V 5900 1700 50  0001 C CNN
+F 2 "footprint-lib:LED_0805_2012Metric" V 5900 1700 50  0001 C CNN
 F 3 "" V 5900 1700 50  0001 C CNN
 	1    5900 1700
@@
 F 0 "D2" V 5950 2550 50  0000 R CNN
 F 1 "LED_GREEN,0805" V 5900 2550 50  0000 R CNN
-F 2 "LED_SMD:LED_0805_2012Metric_Pad1.15x1.40mm_HandSolder" V 5900 2650 50  0001 C CNN
+F 2 "footprint-lib:LED_0805_2012Metric" V 5900 2650 50  0001 C CNN
 F 3 "" V 5900 2650 50  0001 C CNN
 	1    5900 2650
@@
 F 0 "D3" V 5950 3450 50  0000 R CNN
 F 1 "LED_GREEN,0805" V 5900 3450 50  0000 R CNN
-F 2 "LED_SMD:LED_0805_2012Metric_Pad1.15x1.40mm_HandSolder" V 5900 3550 50  0001 C CNN
+F 2 "footprint-lib:LED_0805_2012Metric" V 5900 3550 50  0001 C CNN
 F 3 "" V 5900 3550 50  0001 C CNN
 	1    5900 3550
@@
 F 0 "D4" V 5950 4350 50  0000 R CNN
 F 1 "LED_GREEN,0805" V 5900 4350 50  0000 R CNN
-F 2 "LED_SMD:LED_0805_2012Metric_Pad1.15x1.40mm_HandSolder" V 5900 4450 50  0001 C CNN
+F 2 "footprint-lib:LED_0805_2012Metric" V 5900 4450 50  0001 C CNN
 F 3 "" V 5900 4450 50  0001 C CNN
 	1    5900 4450
